File: KiCad/NixieTubeSchematic/DS3231_Real_Time_Clock.kicad_sch (KiCad schematic)
At the start: 16 parts, among them J1 Conn_01x02_Pin, U2 AT24CS32-SSHM, U3 DS3231MZ

Commit message: Small changes
Connections:
- net I2C1_SCL: no longer RN2.1 (R1.1), RN2.2 (R2.1), U2.5 (SDA), U3.7 (SDA)
- new net I2C1_SDA: U2.5 (SDA), U3.7 (SDA)
- no-connect marks 1 -> 4
Other:
- note removed: "CHECK PULL UP ON I2C MCU SIDE!"
- moved on the sheet: BT1, C1, C2, C3, C4, C5, D1, J1, R2, R3, R4, R5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
